File: untitled.kicad_sch (KiCad schematic)
At the start: 16 parts, among them SW1 SW_Push, U1 STM32G474CBTx, Y1 Crystal_GND24, Y2 Crystal

Commit message: Added differential lines and usb connect
Parts:
- added R1: 10k, symbol Device:R
- added SW2: SW_Push, symbol Switch:SW_Push
- U1: value STM32G474CBTx -> STM32G474CBT6 LQFP-48
Connections:
- net +3.3V: now also SW2.1
- net GND: now also R1.2
- net D-: now reaches U1.33 (PA11)
- net D+: now reaches U1.34 (PA12)
- net SWDIO: now reaches U1.37 (PA13)
- net SWCLK: now reaches U1.38 (PA14)
- net at U1.45 (PB8): now also R1.1, SW2.2

Commit message: adding can IC
Connections:
- net CAN_RX: now reaches U1.26 (PB12)
- net CAN_TX: now reaches U1.27 (PB13)
